File: esp-sme.brd (EAGLE design)
At the start: 58.4 x 33 mm, 30 parts, among them J2 BME280, J3 UART, Q3 NPN, Q4 NPN, Q5 NPN, U2 MIC5504

Commit message: Added boot-pin configuration
Parts:
- added C5: 0.1uF, SparkFun-Capacitors:0603
- added R11, R12, R13, R14, R15: 10k, SparkFun-Resistors:0603
- added S2: FLASH, SparkFun-Switches:TACTILE_SWITCH_SMD_4.6X2.8MM
- moved J3 2.13 mm to (47.9, 1.27)
- moved C3 1.59 mm to (34.9, 28.9)
- moved R10 1.31 mm to (38.7, 31.8)
- moved H1 1.27 mm to (4.08, 2.81)
- moved H2 1.27 mm to (4.08, 30.2)
- moved C4 1.27 mm to (40.6, 31.8)
- moved S1 1.27 mm to (44.5, 31.8)
- moved H3 1.27 mm to (54.3, 2.81)
- moved H4 1.27 mm to (54.3, 30.2)
Connections:
- net N$10 renamed RESET
- new net FLASH: C5.1, R12.1, S2.3, S2.4, U1.GPIO0
- new net N$11: R11.1, U1.CH_PD
- net 3.3V: now also R11.2, R12.2, R14.2, R15.2
- net GND: now also C5.2, R13.1, S2.1, S2.2
- net I2C_SCL: now also R15.1
- net I2C_SDA: now also R14.1
- net LED_G: now also R13.2
Routing:
- net 3.3V: track 76.0 -> 105.9 mm, vias 3 -> 5
- net FLASH: track 0.00 -> 14.9 mm
- net I2C_SCL: track 35.1 -> 39.5 mm
- net I2C_SDA: track 19.1 -> 22.7 mm, vias 0 -> 1
- net N$11: track 0.00 -> 3.45 mm
- net UART_TX: track 6.06 -> 7.57 mm
- net UART_RX: track 34.2 -> 35.7 mm
- net RESET: track 16.5 -> 17.1 mm
Other:
- board size 58.4 x 33 mm -> 58.4 x 35.6 mm
